File: footsquare/footsquaregroundplane.kicad_pcb (KiCad board)
At the start: 2 copper layers, 10 parts, among them J1 USB_B, SW1 RotaryEncoder_Switch, U1 Trill_Craft, U2 Teensy-LC

Commit message: new version with encoder and ground plane
-ground plane added
-encoder added
-outline added
Parts:
- moved REF** 4.80 mm to (249.2, 40.2)
Connections:
- REF** pad 1: Net-(U1-Pad32) -> Net-(J1-Pad4) (x2)
- SW1 pad C: Net-(U1-Pad32) -> Net-(J1-Pad4)
- SW1 pad MP: (no net) -> Net-(J1-Pad4)
- SW1 pad S2: Net-(U1-Pad32) -> Net-(J1-Pad4)
- U1 pad 32: Net-(U1-Pad32) -> Net-(J1-Pad4)
- U2 pad 32: Net-(U1-Pad32) -> Net-(J1-Pad4)
Routing:
- net Net-(U1-Pad32): track 280.1 -> 0.00 mm, vias 1 -> 0
- net Net-(J1-Pad4): track 69.1 -> 9.18 mm
- net Net-(R1-Pad2): track 187.5 -> 182.7 mm
- net Net-(R1-Pad1): track 223.8 -> 221.1 mm
- net Net-(R2-Pad2): track 180.1 -> 178.1 mm
- added copper zone on F.Cu, net Net-(J1-Pad4)
Other:
- board outline added: 279 x 313.8 mm
